File: 2QC+2FSM/2QC+2FSM.kicad_sch (KiCad schematic)
At the start: 33 parts, among them J2 Screw_Terminal_01x04, U4 Teensy4.1, x1 TP_X1, x2 TP_X2, y1 TP_Y1, y2 TP_Y2

Commit message: board layout
Parts:
- FSM1, FSM2: symbol FSM:3220-10-0100-00 -> Connector_Generic_MountingPin:Conn_01x10_MountingPin
- R13, R14: value 1200 -> 2700; LCSC C114526 -> C2907305
- R17: value 300 -> 1000; LCSC C17617 -> C95781
Connections:
- no-connect marks 50 -> 56
