File: 2QC+2FSM/3channels_opamps.kicad_sch (KiCad schematic)
At the start: 50 parts, among them U2 LM4040DBZ-2.0, U8 LM4040DBZ-2.0

Commit message: board layout
Other:
- title: (none) -> X,Y,Sum conversion to 0-3.3V
Changed lines of the file:
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@@
 	(generator_version "9.0")
 	(paper "A4")
+	(title_block
+		(title "X,Y,Sum conversion to 0-3.3V")
+		(date "2025-09-09")
+	)
 	(junction
 		(at 149.86 114.3)
@@
 		)
 	)
-	(label "sum_stage2"
-		(at 170.18 139.7 0)
-		(effects
-			(font
-				(size 1.27 1.27)
-			)
-			(justify left bottom)
-		)
-	)
 	(label "y_stage1"
 		(at 120.65 88.9 0)
@@
 		)
 	)
-	(label "x+"
-		(at 55.88 44.45 0)
-		(effects
-			(font
-				(size 1.27 1.27)
-			)
-			(justify left bottom)
-		)
-	)
-	(label "y_stage2"
-		(at 157.48 86.36 0)
-		(effects
-			(font
-				(size 1.27 1.27)
-			)
-			(justify left bottom)
-		)
-	)
-	(label "x_stage2"
-		(at 158.75 38.1 0)
-		(effects
-			(font
-				(size 1.27 1.27)
-			)
-			(justify left bottom)
-		)
-	)
 	(label "x_stage1"
 		(at 115.57 40.64 0)
@@
 		)
 	)
-	(label "sum"
-		(at 58.42 144.78 0)
-		(effects
-			(font
-				(size 1.27 1.27)
-			)
-			(justify left bottom)
-		)
-	)
 	(label "sum_stage1"
 		(at 120.65 142.24 0)
@@
 		)
 	)
-	(label "y+"
-		(at 67.31 92.71 0)
-		(effects
-			(font
-				(size 1.27 1.27)
-			)
-			(justify left bottom)
-		)
-	)
 	(hierarchical_label "x_out"
 		(shape output)
@@
 	)
 	(symbol
-		(lib_id "power:GND")
-		(at 83.82 33.02 0)
-		(unit 1)
-		(exclude_from_sim no)
-		(in_bom yes)
-		(on_board yes)
-		(dnp no)
-		(fields_autoplaced yes)
-		(property "Reference" "#PWR01"
-			(at 83.82 39.37 0)
-			(effects
-				(font
-					(size 1.27 1.27)
-				)
-				(hide yes)
-			)
-		)
-		(property "Value" "GND"
-			(at 83.82 38.1 0)
-			(effects
-				(font
-					(size 1.27 1.27)
-				)
-			)
-		)
-		(property "Footprint" ""
-			(at 83.82 33.02 0)
-			(effects
-				(font
-					(size 1.27 1.27)
-				)
-				(hide yes)
-			)
-		)
-		(property "Datasheet" ""
-			(at 83.82 33.02 0)
-			(effects
-				(font
-					(size 1.27 1.27)
-				)
-				(hide yes)
-			)
-		)
-		(property "Description" "Power symbol creates a global label with name \"GND\" , ground"
-			(at 83.82 33.02 0)
-			(effects
-				(font
-					(size 1.27 1.27)
-				)
-				(hide yes)
-			)
-		)
-		(pin "1"
-		)
-		(instances
-			(project "2QC+2FSM"
-				(path "/300135d4-a613-4bb1-9425-decc05476821/20600565-84ba-4a93-a38a-83c9dfd701b3"
-					(reference "#PWR01")
-					(unit 1)
-				)
-				(path "/300135d4-a613-4bb1-9425-decc05476821/8f83d0db-1814-4199-b9bf-27ad6d9898ee"
-					(reference "#PWR063")
-					(unit 1)
-				)
-			)
-		)
-	)
-	(symbol
 		(lib_id "JLCPCB-Capacitors:0603,100nF")
 		(at 151.13 76.2 90)
@@
 					(unit 1)
 				)
+			)
+		)
+	)
+	(symbol
+		(lib_id "power:GND")
+		(at 83.82 33.02 0)
+		(unit 1)
+		(exclude_from_sim no)
+		(in_bom yes)
+		(on_board yes)
+		(dnp no)
+		(fields_autoplaced yes)
+		(property "Reference" "#PWR01"
+			(at 83.82 39.37 0)
+			(effects
+				(font
+					(size 1.27 1.27)
+				)
+				(hide yes)
+			)
+		)
+		(property "Value" "GND"
+			(at 83.82 38.1 0)
+			(effects
+				(font
+					(size 1.27 1.27)
+				)
+			)
+		)
+		(property "Footprint" ""
+			(at 83.82 33.02 0)
+			(effects
+				(font
+					(size 1.27 1.27)
+				)
+				(hide yes)
+			)
+		)
+		(property "Datasheet" ""
+			(at 83.82 33.02 0)
+			(effects
+				(font
+					(size 1.27 1.27)
+				)
+				(hide yes)
+			)
+		)
+		(property "Description" "Power symbol creates a global label with name \"GND\" , ground"
+			(at 83.82 33.02 0)
+			(effects
+				(font
+					(size 1.27 1.27)
+				)
+				(hide yes)
+			)
+		)
+		(pin "1"
+		)
+		(instances
+			(project ""
+				(path "/300135d4-a613-4bb1-9425-decc05476821/20600565-84ba-4a93-a38a-83c9dfd701b3"
+					(reference "#PWR01")
+					(unit 1)
+				)
+				(path "/300135d4-a613-4bb1-9425-decc05476821/8f83d0db-1814-4199-b9bf-27ad6d9898ee"
+					(reference "#PWR063")
+					(unit 1)
+				)
