File: 2QC+2FSM/2QC+2FSM.kicad_pcb (KiCad board)
At the start: 2 copper layers, 133 parts, among them J2 Screw_Terminal_01x04, U2 LM4040DBZ-2.0, U4 Teensy4.1, U7 LM4040DBZ-2.0, U8 LM4040DBZ-2.0, U9 LM4040DBZ-2.0, x1 TP_X1, x2 TP_X2, y1 TP_Y1, y2 TP_Y2

Commit message: board layout
Parts:
- R13, R14: value 1200 -> 2700
- R17: value 300 -> 1000
- moved TP_DIN2 157.9 mm to (111.7, 219.6)
- moved TP_EN2 151.1 mm to (104.6, 219.5)
- moved TP_EN1 149.5 mm to (104.9, 212.8)
- moved U4 141.7 mm to (167.6, 192.0), turned to 90 degrees
- moved GND3 139.5 mm to (127.0, 216.8)
- moved TP_SYNC2 136.4 mm to (118.8, 219.5)
- moved TP_SYNC1 134.9 mm to (118.9, 212.9)
- moved TP_DIN1 126.3 mm to (111.7, 212.9)
- moved GND5 112.9 mm to (135.8, 201.6)
- moved H2 106.6 mm to (187.3, 246.0)
- moved FSM2 106.4 mm to (74.5, 234.1), turned to -90 degrees
- moved sum2 101.5 mm to (105.5, 187.7)
- moved H4 98.9 mm to (56.4, 246.0)
- moved FSM1 98.1 mm to (75.0, 213.9), turned to -90 degrees
- moved QC2 90.1 mm to (86.4, 153.5)
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Routing:
- net -15V: track 12.6 -> 468.9 mm, vias 0 -> 26
- net +15V: track 13.4 -> 429.9 mm, vias 0 -> 16
- net GND: track 0.00 -> 340.5 mm, vias 0 -> 12
- net +5V: track 0.00 -> 297.7 mm, vias 0 -> 27
- net /FCLK_X: track 0.00 -> 155.1 mm, vias 0 -> 5
- net /DIN: track 0.00 -> 148.9 mm, vias 0 -> 5
- net /EN2: track 0.00 -> 147.1 mm
- net /FCLK_Y: track 0.00 -> 142.0 mm, vias 0 -> 3
- net /x1_out: track 14.3 -> 156.2 mm, vias 0 -> 1
- net /EN1: track 0.00 -> 128.1 mm, vias 0 -> 6
- net /SYNC2: track 0.00 -> 127.8 mm, vias 0 -> 2
- net /SCLK: track 0.00 -> 122.9 mm, vias 0 -> 5
- net /y1_out: track 14.5 -> 133.3 mm, vias 0 -> 1
- net /SYNC1: track 0.00 -> 116.0 mm, vias 0 -> 4
- net /sum1_out: track 14.8 -> 115.7 mm, vias 0 -> 2
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Other:
- board outline added: 146.3 x 210.1 mm
- board text added: "+-10V"
- board text added: "+15V"
- board text added: "+5V"
- board text added: "-15V"
- board text added: "0>-3.3V"
- board text added: "0>10V"
- board text added: "0>3.3V"
- board text added: "Did you turn it on?"
- board text added: "FSM 1"
- board text added: "FSM 2"
- board text added: "GND"
- board text added: "QC1"
- board text added: "QC1 INPUT"
- board text added: "QC1 SCALING"
- board text added: "QC2"
- board text added: "QC2 INPUT"
- board text added: "QC2 SCALING"
- board text added: "QUADCELL 1"
- board text added: "QUADCELL 2"
- board text added: "SPI for FSM1,2"
- board text added: "SUM"
- board text added: "SUM_{1}"
- board text added: "Teensy Pins 5 - EN1 (Enable FSM1) 6 - EN2 (Enable FSM2) 7 - SYNC1 (CS FSM1) 8 - SYNC2 (CS FSM2) 9 - FCLK X 10 - FCLK Y 11 - DIN (fsm data) 13 - SCLK (SPI clock) 14 - X1 (QC1 x) 15 - Y1 (QC1 y) 16 - Sum1 (QC1 Sum) 17 - X2 (QC2 x) 18 - Y2 (QC2 y) 19 - SUM2 (QC2)"
- board text added: "X+"
- board text added: "X_{1}"
- board text added: "Y+"
- board text added: "Y_{1}"

Commit message: added text and modified layout
Parts:
- moved FSM2 44.1 mm to (116.0, 219.2), turned to 0 degrees
- moved GND3 40.2 mm to (89.2, 203.2)
- moved TP_EN2 25.5 mm to (130.1, 218.1)
- moved TP_DIN2 24.3 mm to (136.0, 218.2)
- moved TP_SYNC2 23.9 mm to (142.7, 218.4)
- moved H2 23.5 mm to (183.0, 222.9)
- moved H4 22.8 mm to (60.2, 223.5)
- moved TP_SYNC1 20.4 mm to (99.1, 217.7)
- moved TP_DIN1 20.3 mm to (92.0, 217.7)
- moved TP_EN1 19.5 mm to (86.0, 217.7)
- moved D3 11.4 mm to (173.6, 83.1)
- moved R13 11.4 mm to (166.9, 70.5)
- moved R14 11.4 mm to (167.2, 76.3)
- moved R17 11.4 mm to (167.2, 83.1)
- moved D1 11.4 mm to (173.6, 70.7)
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- renumbered x1 to x_{1}
Routing:
- net /EN2: track 147.1 -> 84.0 mm
- net /SYNC2: track 127.8 -> 67.6 mm
- net /FCLK_X: track 155.1 -> 114.5 mm, vias 5 -> 2
- net GND: track 340.5 -> 304.9 mm, vias 12 -> 18
- net /DIN: track 148.9 -> 116.0 mm, vias 5 -> 1
- net +5V: track 297.7 -> 328.6 mm, vias 27 -> 28
- net /FCLK_Y: track 142.0 -> 114.1 mm, vias 3 -> 2
- net /SCLK: track 122.9 -> 99.0 mm, vias 5 -> 2
- net /EN1: track 128.1 -> 111.5 mm, vias 6 -> 2
- net /SYNC1: track 116.0 -> 107.4 mm, vias 4 -> 3
- net -15V: track 468.9 -> 470.2 mm
- net +15V: track 429.9 -> 430.7 mm
Other:
- board size 146.3 x 210.1 mm -> 132.5 x 186.2 mm
- board text added: "Data sent over SPI to Mirrorcle FSM Driver"
- board text added: "Did you plug it in?"
- board text added: "POWER IN"
- board text added: "QUADCELL 1 SCALING"
- board text added: "QUADCELL 2 SCALING"
- board text added: "SUM_{2}"
- board text added: "Teensy 4.1"
- board text added: "Teensy 4.1 control of 2 FSM, 2 QC Precision Pointing Testbed Oct 2025 Paige Forester paigefor@mit.edu"
- board text added: "X,Y from +-10V into 0-3.3V SUM from 0-10V into 0-3.3V"
- board text added: "X_{2}"
- board text added: "Y_{2}"
- board text added: "stage1:sum_{1}"
- board text added: "stage1:sum_{2}"
- board text added: "stage1:x_{1}"
- board text added: "stage1:x_{2}"
- board text added: "stage1:y_{1}"
- board text added: "stage1:y_{2}"
- board text added: "stage2:sum_{1}"
- board text added: "stage2:sum_{2}"
- board text added: "stage2:x_{1}"
- board text added: "stage2:x_{2}"
- board text added: "stage2:y_{1}"
- board text added: "stage2:y_{2}"
- board text added: "x_{2}"
- board text added: "y_{1}"
- board text added: "y_{2}"
- board text removed: "Did you turn it on?"
- board text removed: "QC1 INPUT"
- board text removed: "QC1 SCALING"
- board text removed: "QC2 INPUT"
- board text removed: "QC2 SCALING"
